File: Hardware_UniversalRemote/Hardware_UniversalRemote.kicad_sch (KiCad schematic)
At the start: 56 parts, among them J1 USB_B_Micro, Q1 S8050, Q2 S8050, Q3 S8050, Q4 S8050, Q5 S8050, Q6 S8050, SW1 SW_Push, SW2 SW_Push, SW3 SW_Push, U1 ESP32-WROOM-32U, U2 LM1117T-3.3, U3 HS0038B, U4 CH340C

Commit message: add capacitor footprint
Parts:
- C1, C10, C11, C12, C4, C8, C9: footprint (none) -> Capacitor_THT:C_Disc_D3.4mm_W2.1mm_P2.50mm
- C3, C5: footprint (none) -> Capacitor_THT:CP_Radial_D4.0mm_P2.00mm
- C7: footprint (none) -> Capacitor_THT:CP_Radial_D5.0mm_P2.00mm
- CB1: footprint (none) -> Fuse:Fuse_1812_4532Metric_Pad1.30x3.40mm_HandSolder
Changed lines of the file:
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@@
 			)
 		)
-		(property "Footprint" ""
+		(property "Footprint" "Fuse:Fuse_1812_4532Metric_Pad1.30x3.40mm_HandSolder"
 			(at 55.88 29.21 0)
 			(effects
@@
 			)
 		)
-		(property "Footprint" ""
+		(property "Footprint" "Capacitor_THT:C_Disc_D3.4mm_W2.1mm_P2.50mm"
 			(at 234.95 147.32 0)
 			(effects
@@
 			)
 		)
-		(property "Footprint" ""
+		(property "Footprint" "Capacitor_THT:C_Disc_D3.4mm_W2.1mm_P2.50mm"
 			(at 80.01 96.52 0)
 			(effects
@@
 			)
 		)
-		(property "Footprint" ""
+		(property "Footprint" "Capacitor_THT:CP_Radial_D5.0mm_P2.00mm"
 			(at 148.59 173.99 0)
 			(effects
@@
 			)
 		)
-		(property "Footprint" ""
+		(property "Footprint" "Capacitor_THT:C_Disc_D3.4mm_W2.1mm_P2.50mm"
 			(at 153.67 90.17 0)
 			(effects
@@
 			)
 		)
-		(property "Footprint" ""
+		(property "Footprint" "Capacitor_THT:C_Disc_D3.4mm_W2.1mm_P2.50mm"
 			(at 234.95 110.49 0)
 			(effects
@@
 			)
 		)
-		(property "Footprint" ""
+		(property "Footprint" "Capacitor_THT:CP_Radial_D4.0mm_P2.00mm"
 			(at 76.2 85.09 0)
 			(effects
@@
 			)
 		)
-		(property "Footprint" ""
+		(property "Footprint" "Capacitor_THT:C_Disc_D3.4mm_W2.1mm_P2.50mm"
 			(at 153.67 85.09 0)
 			(effects
@@
 			)
 		)
-		(property "Footprint" ""
+		(property "Footprint" "Capacitor_THT:C_Disc_D3.4mm_W2.1mm_P2.50mm"
 			(at 234.95 86.36 0)
 			(effects
@@
 			)
 		)
-		(property "Footprint" ""
+		(property "Footprint" "Capacitor_THT:C_Disc_D3.4mm_W2.1mm_P2.50mm"
 			(at 34.29 118.11 0)
 			(effects
@@
 			)
 		)
-		(property "Footprint" ""
+		(property "Footprint" "Capacitor_THT:CP_Radial_D4.0mm_P2.00mm"
 			(at 83.82 85.09 0)
 			(effects

Commit message: add net list
Parts:
- removed C9: 0.1uF, Capacitor_THT:C_Disc_D3.4mm_W2.1mm_P2.50mm, symbol Device:C_Small
- D1: footprint (none) -> Diode_THT:D_DO-41_SOD81_P7.62mm_Horizontal
- D2: footprint (none) -> LED_THT:LED_D3.0mm
- D3, D4, D5, D6, D7, D8, D9: footprint (none) -> LED_THT:LED_D5.0mm
- J1: footprint (none) -> Connector_USB:USB_Micro-B_Wuerth_629105150521
- R1, R11, R13, R14, R2, R3, R4, R5, R7, R8, R9: footprint (none) -> Resistor_THT:R_Axial_DIN0207_L6.3mm_D2.5mm_P7.62mm_Horizontal
- R10, R12, R15, R6: footprint (none) -> Resistor_THT:R_Axial_DIN0414_L11.9mm_D4.5mm_P15.24mm_Horizontal
- SW1, SW2, SW3: footprint (none) -> Button_Switch_THT:SW_TH_Tactile_Omron_B3F-10xx
- TP1, TP2, TP3, TP4, TP5: footprint (none) -> TestPoint:TestPoint_Pad_D2.5mm
- U3: footprint (none) -> Package_TO_SOT_THT:TO-92_Inline_Wide
- renumbered C11 to C10, C12 to C11, C10 to C9
Connections:
- net +3.3V: now also C8.1, U4.16 (VCC), U4.4 (V3)
- net +5V: no longer C8.1, U4.16 (VCC)
Other:
- moved on the sheet: C8

Commit message: add first pcb layout
Parts:
- added Q2: BSS138, Package_TO_SOT_SMD:SOT-23, symbol Transistor_FET:BSS138
- added R5: 10k, Resistor_THT:R_Axial_DIN0207_L6.3mm_D2.5mm_P7.62mm_Horizontal, symbol Device:R
- added R7: 5.6R, Resistor_THT:R_Axial_DIN0414_L11.9mm_D4.5mm_P15.24mm_Horizontal, symbol Device:R
- R6: value 12R -> 5.6R
- renumbered Q2 to Q3, Q3 to Q4, Q4 to Q5, Q5 to Q6, Q6 to Q7, R8 to R10, R9 to R11, R10 to R12, R11 to R13, R12 to R14, R13 to R15, R14 to R16, R15 to R17, R4 to R3, R3 to R4, R5 to R8, R7 to R9
Connections:
- net +3.3V: now also R8.2, Q2.1 (G)
- net +5V: now also R3.1, R5.2; no longer R3.2, R8.1
- net GND: now also C6.2, D1.2 (A), J1.5 (GND), J1.6 (Shield), TP4.1, U2.1 (GND)
- net IO16: now also R8.1, Q2.2 (S); no longer R8.2, U3.1 (IR)
- net at C7.1, U3.3 (VCC): now also R3.2; no longer R3.1
- net at D3.2 (A): now also R7.2; no longer R6.2
- new net: Q2.3 (D), R5.1, U3.1 (IR)
- new net: R6.2, R7.1
Other:
- moved on the sheet: C7, D3, R3, R8, U3
