File: Hardware_UniversalRemote/Hardware_UniversalRemote.kicad_pcb (KiCad board)
At the start: 2 copper layers, 140 x 140 mm, 55 parts, among them J1 USB_B_Micro, Q1 S8050, Q2 S8050, Q3 S8050, Q4 S8050, Q5 S8050, Q6 S8050, SW1 SW_Push, SW2 SW_Push, SW3 SW_Push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

Commit message: add first pcb layout
Parts:
- added Q7: S8050, Package_TO_SOT_THT:TO-92_Inline, F.Cu at (72.6, 122.2)
- added R16: 10k, Resistor_THT:R_Axial_DIN0207_L6.3mm_D2.5mm_P7.62mm_Horizontal, F.Cu at (136.4, 132.1)
- added R17: 5.6R, Resistor_THT:R_Axial_DIN0414_L11.9mm_D4.5mm_P15.24mm_Horizontal, F.Cu at (60.6, 103.7)
- D3, D4, D5, D6, D7, D8, D9: moved to F.Cu
- Q2: value S8050 -> BSS138; footprint Package_TO_SOT_THT:TO-92_Inline -> Package_TO_SOT_SMD:SOT-23
- R10: value 5.6R -> 10k; footprint Resistor_THT:R_Axial_DIN0414_L11.9mm_D4.5mm_P15.24mm_Horizontal -> Resistor_THT:R_Axial_DIN0207_L6.3mm_D2.5mm_P7.62mm_Horizontal
- R11, R3: value 1k -> 10k
- R14: value 10k -> 5.6R; footprint Resistor_THT:R_Axial_DIN0207_L6.3mm_D2.5mm_P7.62mm_Horizontal -> Resistor_THT:R_Axial_DIN0414_L11.9mm_D4.5mm_P15.24mm_Horizontal
- R15: value 5.6R -> 1k; footprint Resistor_THT:R_Axial_DIN0414_L11.9mm_D4.5mm_P15.24mm_Horizontal -> Resistor_THT:R_Axial_DIN0207_L6.3mm_D2.5mm_P7.62mm_Horizontal
- R4, R9: value 10k -> 1k
- R6: value 12R -> 5.6R
- R7: value 1k -> 5.6R; footprint Resistor_THT:R_Axial_DIN0207_L6.3mm_D2.5mm_P7.62mm_Horizontal -> Resistor_THT:R_Axial_DIN0414_L11.9mm_D4.5mm_P15.24mm_Horizontal
- U2: footprint Package_TO_SOT_THT:TO-220-3_Vertical -> Package_TO_SOT_THT:TO-220-3_Horizontal_TabDown
- moved TP3 191.3 mm to (46.2, 136.8)
- moved TP5 164.4 mm to (71.9, 46.9)
- moved C3 160.8 mm to (54.6, 144.1), turned to 90 degrees
- moved C2 159.9 mm to (90.3, 44.7), turned to 90 degrees
- moved TP1 158.1 mm to (93.9, 154.8)
- moved C5 158.0 mm to (54.6, 137.9), turned to 90 degrees
- moved C1 151.0 mm to (54.3, 151.2), turned to 90 degrees
- moved C4 140.4 mm to (61.8, 145.2), turned to 90 degrees
- moved SW1 124.5 mm to (115.4, 141.9), turned to 90 degrees
- moved TP4 123.1 mm to (115.5, 36.4)
- moved R15 123.0 mm to (81.0, 121.6), turned to 90 degrees
- moved SW2 111.6 mm to (126.3, 142.7), turned to 90 degrees
- moved R6 110.0 mm to (99.4, 117.8)
- moved C7 105.0 mm to (136.7, 118.9), turned to 90 degrees
- moved Q6 99.0 mm to (95.9, 76.6), turned to 180 degrees
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Connections:
- C6 pad 2: Net-(D1-A) -> GND
- D1 pad 2: Net-(D1-A) -> GND
- J1 pad 5: Net-(D1-A) -> GND
- J1 pad 6: Net-(D1-A) -> GND
- Q2 pad 1: GND -> +3.3V
- Q2 pad 2: Net-(Q2-B) -> /IO16
- Q2 pad 3: Net-(D5-K) -> Net-(Q2-D)
- Q3 pad 1: /RTS -> GND
- Q3 pad 3: /EN -> Net-(D5-K)
- Q4 pad 1: /DTR -> /RTS
- Q4 pad 3: /IO0 -> /EN
- Q5 pad 1: GND -> /DTR
- Q5 pad 3: Net-(D7-K) -> /IO0
- Q6 pad 3: Net-(D9-K) -> Net-(D7-K)
- R10 pad 1: +5V -> /DTR
- R10 pad 2: Net-(D4-A) -> Net-(Q4-B)
- R11 pad 1: /IO4 -> /RTS
- R12 pad 2: Net-(D6-A) -> Net-(D4-A)
- R14 pad 1: +3.3V -> +5V
- R14 pad 2: /IO13 -> Net-(D6-A)
- R15 pad 1: +5V -> /IO4
- R15 pad 2: Net-(D8-A) -> Net-(Q7-B)
- R3 pad 1: /IO4 -> +5V
- R3 pad 2: Net-(Q1-B) -> Net-(U3-VCC)
- R4 pad 1: Net-(U3-VCC) -> /IO4
- R4 pad 2: +5V -> Net-(Q1-B)
- R5 pad 1: +5V -> Net-(Q2-D)
- R5 pad 2: /IO16 -> +5V
- R6 pad 2: Net-(D3-A) -> Net-(R6-Pad2)
- R7 pad 1: /IO4 -> Net-(R6-Pad2)
- R7 pad 2: Net-(Q2-B) -> Net-(D3-A)
- R8 pad 1: /DTR -> /IO16
- R8 pad 2: Net-(Q3-B) -> +3.3V
- R9 pad 1: /RTS -> /IO4
- R9 pad 2: Net-(Q4-B) -> Net-(Q3-B)
- TP4 pad 1: Net-(D1-A) -> GND
- U2 pad 1: Net-(D1-A) -> GND
- U3 pad 1: /IO16 -> Net-(Q2-D)

Commit message: add first pcb layout version
Parts:
- moved TP3 129.7 mm to (172.5, 107.5)
- moved TP5 124.0 mm to (172.5, 119.5)
- moved TP4 95.9 mm to (172.5, 113.5)
- moved U1 91.0 mm to (136.0, 90.2)
- moved C1 90.5 mm to (120.2, 89.2), turned to 180 degrees
- moved R1 88.8 mm to (112.6, 85.0), turned to 0 degrees
- moved C5 88.0 mm to (113.7, 72.8)
- moved C4 87.3 mm to (120.1, 80.2)
- moved C3 86.8 mm to (113.4, 80.2)
- moved R9 73.0 mm to (80.9, 143.9), turned to 90 degrees
- moved R12 67.1 mm to (60.4, 90.9)
- moved R4 60.4 mm to (68.5, 143.7), turned to 90 degrees
- moved U3 58.2 mm to (144.2, 165.1), turned to 180 degrees
- moved R13 55.8 mm to (53.0, 119.0), turned to 0 degrees
- moved SW1 55.5 mm to (170.4, 134.6), turned to -90 degrees
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Connections:
- C11 pad 1: /IO13 -> /IO16
- Q2 pad 2: /IO16 -> /IO13
- R16 pad 2: /IO13 -> /IO16
- R8 pad 1: /IO16 -> /IO13
- SW3 pad 1: /IO13 -> /IO16
- TP2 pad 1: /IO16 -> /IO13
Routing:
- net GND: track 0.00 -> 114.7 mm
- net +5V: track 0.00 -> 82.8 mm
- net Net-(D9-K): track 0.00 -> 54.8 mm
- net Net-(D3-A): track 0.00 -> 48.2 mm
- net Net-(D3-K): track 0.00 -> 45.6 mm
- net Net-(D4-A): track 0.00 -> 44.5 mm
- net /IO4: track 0.00 -> 43.6 mm
- net Net-(D8-A): track 0.00 -> 43.0 mm
- net /RXD0: track 0.00 -> 42.1 mm
- net /TXD0: track 0.00 -> 40.7 mm
- net Net-(D6-A): track 0.00 -> 39.1 mm
- net +3.3V: track 0.00 -> 35.3 mm
- net /EN: track 0.00 -> 34.8 mm
- net Net-(D5-K): track 0.00 -> 33.0 mm
- net Net-(D7-K): track 0.00 -> 32.7 mm
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
Commit message: improve layout
Parts:
- D3: moved to B.Cu
- D4, D5, D6, D7, D8, D9: footprint LED_THT:LED_D5.0mm -> LED_THT:LED_D5.0mm_Horizontal_O3.81mm_Z3.0mm; moved to B.Cu
- moved D1 25.3 mm to (136.2, 51.0)
- moved U4 20.5 mm to (112.0, 62.5)
- moved D5 9.66 mm to (112.3, 126.0), turned to 180 degrees
- moved D9 9.49 mm to (117.7, 121.4), turned to -120 degrees
- moved D4 9.39 mm to (105.6, 123.6), turned to 120 degrees
- moved D8 9.04 mm to (116.4, 114.4), turned to -60 degrees
- moved D7 8.93 mm to (104.3, 116.6), turned to 60 degrees
- moved D6 8.75 mm to (109.7, 112.0), turned to 0 degrees
- moved CB1 7.01 mm to (99.0, 57.5)
- moved C5 6.38 mm to (120.0, 73.5)
- moved U1 2.62 mm to (137.2, 92.6)
- moved C8 2.50 mm to (132.8, 57.0), turned to 180 degrees
- moved J1 0.15 mm to (110.9, 52.8), turned to 180 degrees
Routing:
- net GND: track 114.7 -> 0.00 mm
- net +5V: track 82.8 -> 0.00 mm
- net Net-(D9-K): track 54.8 -> 0.00 mm
- net Net-(D3-A): track 48.2 -> 0.00 mm
- net Net-(D3-K): track 45.6 -> 0.00 mm
- net Net-(D4-A): track 44.5 -> 0.00 mm
- net /IO4: track 43.6 -> 0.00 mm
- net Net-(D8-A): track 43.0 -> 0.00 mm
- net /RXD0: track 42.1 -> 0.00 mm
- net /TXD0: track 40.7 -> 0.00 mm
- net Net-(D6-A): track 39.1 -> 0.00 mm
- net +3.3V: track 35.3 -> 0.00 mm
- net /EN: track 34.8 -> 0.00 mm
- net Net-(D5-K): track 33.0 -> 0.00 mm
- net Net-(D7-K): track 32.7 -> 0.00 mm
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
Commit message: modify layout
Parts:
- D4, D5, D6, D7, D8, D9: footprint LED_THT:LED_D5.0mm_Horizontal_O3.81mm_Z3.0mm -> LED_THT:LED_D5.0mm
- moved C10 198.1 mm to (-38.4, 161.0)
- moved C7 198.1 mm to (-49.5, 162.8)
- moved C9 198.1 mm to (-27.1, 161.0)
- moved Q2 198.1 mm to (-56.2, 140.5)
- moved R3 198.1 mm to (-57.0, 157.0)
- moved R5 198.1 mm to (-49.4, 152.4)
- moved R8 198.1 mm to (-49.4, 147.8)
- moved SW1 198.1 mm to (-27.1, 150.2)
- moved SW2 198.1 mm to (-38.4, 150.2)
- moved TP2 198.1 mm to (-32.5, 139.1)
- moved TP3 198.1 mm to (-25.0, 123.1)
- moved TP4 198.1 mm to (-25.0, 129.1)
- moved TP5 198.1 mm to (-25.0, 135.1)
- moved U3 194.2 mm to (-47.4, 133.5), turned to -90 degrees
- moved C11 161.2 mm to (-21.6, 61.5)
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Connections:
- J1 pad 4: unconnected-(J1-ID-Pad4) -> GND
Routing:
- net GND: track 0.00 -> 96.6 mm
- net +5V: track 0.00 -> 93.7 mm
- net /IO4: track 0.00 -> 64.7 mm
- net /TXD0: track 0.00 -> 55.9 mm, vias 0 -> 2
- net /RXD0: track 0.00 -> 44.1 mm, vias 0 -> 2
- net Net-(D3-A): track 0.00 -> 32.6 mm
- net Net-(D8-A): track 0.00 -> 28.4 mm
- net Net-(D6-A): track 0.00 -> 24.0 mm
- net Net-(D4-A): track 0.00 -> 22.5 mm
- net +3.3V: track 0.00 -> 22.3 mm, vias 0 -> 1
- net Net-(D3-K): track 0.00 -> 18.3 mm
- net Net-(J1-VBUS): track 0.00 -> 14.7 mm
- net Net-(D5-K): track 0.00 -> 11.7 mm
- net Net-(D8-K): track 0.00 -> 10.4 mm
- net Net-(Q3-B): track 0.00 -> 9.15 mm
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
Commit message: modify routing
Parts:
- D4, D5, D6, D7, D8, D9: footprint LED_THT:LED_D5.0mm -> LED_THT:LED_D5.0mm_Horizontal_O3.81mm_Z9.0mm
- moved R3 199.6 mm to (142.5, 152.9), turned to 180 degrees
- moved TP4 197.9 mm to (172.5, 116.5)
- moved U3 193.8 mm to (142.6, 171.7), turned to 180 degrees
- moved R5 192.3 mm to (142.5, 165.5), turned to 90 degrees
- moved TP5 191.4 mm to (165.5, 116.8)
- moved Q2 188.5 mm to (130.7, 164.7), turned to -90 degrees
- moved C7 186.1 mm to (136.5, 161.6), turned to 0 degrees
- moved TP3 184.3 mm to (159.2, 116.7)
- moved R8 173.6 mm to (123.9, 158.9), turned to 0 degrees
- moved TP2 158.7 mm to (124.3, 163.8)
- moved SW3 151.8 mm to (94.3, 154.0)
- moved C11 142.3 mm to (94.3, 144.2)
- moved R16 122.7 mm to (87.3, 100.8), turned to 0 degrees
- moved R2 118.1 mm to (83.9, 103.2), turned to -90 degrees
- moved D2 111.4 mm to (83.9, 117.0), turned to 90 degrees
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Routing:
- net GND: track 96.6 -> 395.1 mm
- net /EN: track 0.00 -> 126.3 mm
- net /IO13: track 0.00 -> 107.2 mm, vias 0 -> 2
- net /IO0: track 0.00 -> 78.6 mm, vias 0 -> 1
- net +3.3V: track 22.3 -> 93.8 mm, vias 1 -> 0
- net /IO16: track 0.00 -> 66.6 mm
- net /DTR: track 0.00 -> 38.7 mm
- net /IO4: track 64.7 -> 100.7 mm
- net /IO17: track 0.00 -> 30.4 mm, vias 0 -> 1
- net /RTS: track 0.00 -> 27.9 mm
- net Net-(Q2-D): track 0.00 -> 18.2 mm
- net Net-(Q5-B): track 0.00 -> 15.1 mm
- net Net-(U1-VDD): track 0.00 -> 13.7 mm
- net Net-(Q4-B): track 0.00 -> 13.6 mm
- net Net-(D6-A): track 24.0 -> 13.3 mm
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
Commit message: add trace
Parts:
- moved C4 28.4 mm to (76.5, 105.0), turned to 0 degrees
- moved C3 21.6 mm to (68.3, 107.3), turned to 0 degrees
- moved TP4 20.2 mm to (159.2, 131.7)
- moved C5 19.3 mm to (68.3, 112.3), turned to 0 degrees
- moved R3 16.7 mm to (146.6, 136.8)
- moved U3 16.7 mm to (146.7, 155.6)
- moved C7 16.7 mm to (140.6, 145.5)
- moved Q2 16.7 mm to (134.8, 148.6)
- moved R5 16.7 mm to (146.6, 149.4)
- moved C10 12.5 mm to (74.6, 121.9)
- moved SW2 12.4 mm to (72.5, 132.2)
- moved R8 11.2 mm to (129.7, 149.3), turned to 90 degrees
- moved C9 10.9 mm to (84.7, 121.9)
- moved SW1 10.7 mm to (84.7, 125.8)
- moved TP2 9.97 mm to (129.6, 155.4)
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Connections:
- C3 pad 1: Net-(U1-VDD) -> +3.3V
- C4 pad 1: Net-(U1-VDD) -> +3.3V
- U1 pad 2: Net-(U1-VDD) -> +3.3V
Routing:
- net +3.3V: track 93.8 -> 256.3 mm
- net +5V: track 99.8 -> 153.6 mm, vias 0 -> 1
- net /EN: track 126.3 -> 99.4 mm
- net GND: track 395.1 -> 378.6 mm
- net /TXD0: track 57.9 -> 42.0 mm
- net Net-(U1-VDD): track 13.7 -> 0.00 mm
- net /IO0: track 78.6 -> 66.6 mm
- net Net-(U3-VCC): track 9.39 -> 19.9 mm
- net /IO17: track 30.4 -> 21.4 mm, vias 1 -> 0
- net Net-(D4-A): track 22.5 -> 17.6 mm
- net /RTS: track 27.9 -> 24.5 mm
- net /DTR: track 38.7 -> 35.7 mm
- net Net-(D2-A): track 3.68 -> 6.37 mm
- net Net-(J1-VBUS): track 14.7 -> 16.4 mm
- net /IO13: track 107.2 -> 105.8 mm
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Other:
- board size 140 x 140 mm -> 130 x 130 mm

Commit message: finished second pcb layout
Parts:
- moved TP3 15.3 mm to (144.8, 111.5)
- moved TP5 15.3 mm to (144.8, 119.3)
- moved TP4 15.3 mm to (144.8, 126.5)
Routing:
- net GND: track 378.6 -> 418.8 mm
- net +3.3V: track 256.3 -> 222.6 mm
- net +5V: track 153.6 -> 137.7 mm

Commit message: fix txd/rxd routing for mcu flashing
Connections:
- U4 pad 2: /TXD0 -> /RXD0
- U4 pad 3: /RXD0 -> /TXD0
Routing:
- net GND: track 418.8 -> 432.0 mm
- net /TXD0: track 42.0 -> 40.8 mm
- net /RXD0: track 44.0 -> 44.8 mm
Changed lines of the file:
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@@
 			(layers "F.Cu" "F.Paste" "F.Mask")
 			(roundrect_rratio 0.25)
-			(net 57 "/TXD0")
+			(net 41 "/RXD0")
 			(pinfunction "TXD")
 			(pintype "output")
@@
 			(layers "F.Cu" "F.Paste" "F.Mask")
 			(roundrect_rratio 0.25)
-			(net 41 "/RXD0")
+			(net 57 "/TXD0")
 			(pinfunction "RXD")
 			(pintype "input")
@@
 			(net 48 "/SENSOR_VP")
 			(pinfunction "SENSOR_VP")
-			(pintype "input")
+			(pintype "input+no_connect")
 		)
 		(pad "5" smd rect
@@
 			(net 49 "/SENSOR_VN")
 			(pinfunction "SENSOR_VN")
-			(pintype "input")
+			(pintype "input+no_connect")
 		)
 		(pad "6" smd rect
@@
 	)
 	(segment
+		(start 70.885 97.75)
+		(end 70.885 101.185)
+		(width 0.3)
+		(layer "F.Cu")
+		(net 2)
+	)
+	(segment
 		(start 96 127)
 		(end 96 119.5)
@@
 	)
 	(segment
+		(start 70.885 101.185)
+		(end 73.2 103.5)
+		(width 0.3)
+		(layer "F.Cu")
+		(net 2)
+	)
+	(segment
 		(start 81.8 105.05)
 		(end 79 105.05)
@@
 	)
 	(segment
+		(start 79 105.05)
+		(end 77.45 103.5)
+		(width 0.3)
+		(layer "B.Cu")
+		(net 2)
+	)
+	(segment
 		(start 73.25 110.8)
 		(end 79 105.05)
@@
 	)
 	(segment
+		(start 77.45 103.5)
+		(end 73.2 103.5)
+		(width 0.3)
+		(layer "B.Cu")
+		(net 2)
+	)
+	(segment
 		(start 131.12 98.38)
 		(end 134.38 95.12)
@@
 	)
 	(segment
-		(start 111.55 66.27)
-		(end 111.555 66.275)
+		(start 85.6 85.475)
+		(end 85.35 85.225)
 		(width 0.2)
 		(layer "F.Cu")
@@
 	)
 	(segment
-		(start 85.6 85.475)
-		(end 85.35 85.225)
+		(start 112.8 66.3)
+		(end 112.825 66.275)
 		(width 0.2)
 		(layer "F.Cu")
@@
 	)
 	(segment
-		(start 111.55 64.15)
-		(end 111.55 66.27)
+		(start 112.825 66.275)
+		(end 112.825 64.995)
+		(width 0.2)
+		(layer "F.Cu")
+		(net 41)
+	)
+	(segment
+		(start 112.825 64.995)
+		(end 112 64.17)
 		(width 0.2)
 		(layer "F.Cu")
@@
 	)
 	(via
-		(at 111.55 64.15)
+		(at 112 64.17)
 		(size 0.6)
 		(drill 0.3)
@@
 	)
 	(segment
-		(start 107.9 64.2)
-		(end 111.5 64.2)
+		(start 111.97 64.2)
+		(end 112 64.17)
 		(width 0.2)
 		(layer "B.Cu")
@@
 	)
 	(segment
-		(start 92.17 82.96)
-		(end 89.655 85.475)
+		(start 107.9 64.2)
+		(end 111.5 64.2)
 		(width 0.2)
 		(layer "B.Cu")
@@
 	)
 	(segment
-		(start 111.5 64.2)
-		(end 111.55 64.15)
+		(start 92.17 82.96)
+		(end 89.655 85.475)
 		(width 0.2)
 		(layer "B.Cu")
@@
 	)
 	(segment
+		(start 111.5 64.2)
+		(end 111.97 64.2)
+		(width 0.2)
+		(layer "B.Cu")
+		(net 41)
+	)
+	(segment
 		(start 93.96 82.71)
 		(end 92.465 84.205)
@@
 	)
 	(segment
-		(start 112.8 68.15)
-		(end 112.8 66.3)
+		(start 93.96 72.54)
+		(end 93.96 82.71)
 		(width 0.2)
 		(layer "F.Cu")
@@
 	)
 	(segment
-		(start 93.96 72.54)
-		(end 93.96 82.71)
+		(start 99.45 68.95)
+		(end 99.6 68.8)
 		(width 0.2)
 		(layer "F.Cu")
@@
 	)
 	(segment
-		(start 99.45 68.95)
-		(end 99.6 68.8)
+		(start 111.555 66.275)
+		(end 111.555 67.945)
 		(width 0.2)
 		(layer "F.Cu")
@@
 	)
 	(segment
-		(start 112.8 66.3)
-		(end 112.825 66.275)
+		(start 111.55 66.27)
+		(end 111.555 66.275)
+		(width 0.2)
+		(layer "F.Cu")
+		(net 57)
+	)
+	(segment
+		(start 111.555 67.945)
+		(end 111.62 68.01)
 		(width 0.2)
 		(layer "F.Cu")
@@
 	)
 	(via
-		(at 112.8 68.15)
+		(at 111.62 68.01)
 		(size 0.6)
 		(drill 0.3)
@@
 	)
 	(segment
-		(start 112.15 68.8)
-		(end 112.8 68.15)
+		(start 110.83 68.8)
+		(end 111.62 68.01)
 		(width 0.2)
 		(layer "B.Cu")
@@
 	(segment
 		(start 99.6 68.8)
-		(end 112.15 68.8)
+		(end 110.83 68.8)
 		(width 0.2)
 		(layer "B.Cu")
